Commit message: fix: stabilize option 17 detour simulation

File: src/traymover_robot_description/urdf/traymover_sim.urdf.xacro (robot description, xacro)
@@ -9,11 +9,12 @@
   <xacro:property name="wheel_separation" value="0.455"/>
   <material name="traymover_gray"><color rgba="0.28 0.31 0.34 1"/></material>
-  <material name="traymover_black"><color rgba="0.08 0.08 0.08 1"/></material>
-  <material name="traymover_blue"><color rgba="0.15 0.35 0.85 1"/></material>
+  <material name="traymover_black"><color rgba="0.05 0.06 0.09 1"/></material>
+  <material name="traymover_blue"><color rgba="0.03 0.55 0.95 1"/></material>
+  <material name="traymover_yellow"><color rgba="1.0 0.72 0.0 1"/></material>
   <link name="base_link">
     <inertial><mass value="20.0"/><origin xyz="0 0 0.2"/>
       <inertia ixx="1.0" ixy="0" ixz="0" iyy="1.0" iyz="0" izz="1.0"/>
     </inertial>
-    <visual><origin xyz="0 0 0.2"/><geometry><box size="${body_length} ${body_width} ${body_height}"/></geometry><material name="traymover_gray"/></visual>
+    <visual><origin xyz="0 0 0.2"/><geometry><box size="${body_length} ${body_width} ${body_height}"/></geometry><material name="traymover_blue"/></visual>
     <collision><origin xyz="0 0 0.2"/><geometry><box size="${body_length} ${body_width} ${body_height}"/></geometry></collision>
   </link>
@@ -33,5 +34,5 @@
   <link name="laser">
     <inertial><mass value="0.1"/><inertia ixx="0.0001" ixy="0" ixz="0" iyy="0.0001" iyz="0" izz="0.0001"/></inertial>
-    <visual><geometry><cylinder radius="0.06" length="0.05"/></geometry><material name="traymover_blue"/></visual>
+    <visual><geometry><cylinder radius="0.06" length="0.05"/></geometry><material name="traymover_yellow"/></visual>
     <collision><geometry><cylinder radius="0.06" length="0.05"/></geometry></collision>
   </link>
@@ -67,5 +68,7 @@
           <min_angle>-2.35619449</min_angle><max_angle>2.35619449</max_angle>
         </horizontal></scan>
-        <range><min>0.2</min><max>8.0</max><resolution>0.01</resolution></range>
+        <!-- Keep near-field returns so a stopped robot can still put a
+             blocking box into Nav2's global obstacle layer. -->
+        <range><min>0.05</min><max>8.0</max><resolution>0.01</resolution></range>
       </ray>
     </sensor>
